File: RPi-pHat-Thermocouple.sch (KiCad schematic (older format))
At the start: 54 parts, among them J1 RPi_GPIO, J2 Barrel_Jack_Switch, P1 CONN_01X02, P2 CONN_01X02, P3 CONN_01X02, P6 CONN_01X03, Q1 NUD3124, Q2 BCM857BS, Q3 DMG2305UX, SW1 Write, U1 MAX31850K, U2 MAX31850K, U3 MAX31850K, U4 DS18S20, U5 AT24CS32, U6 LMZ21700, U7 MCP1754ST

Commit message: Variation for generator monitoring application.
Remove buzzer and related; remove Pi Hat EEPROM.

Since the form factor is going to expand a bit beyond the Pi-Hat
specification to enable adding an isolated RS-232/TTL interface for
the Raspberry Pi serial port, we'll remove the parts that are not needed
for the generator-targeted application.
Parts:
- removed BZ1: Buzzer, Buzzer_Beeper-ML:MagneticBuzzer_CUI-CMI-9655S, symbol Device:Buzzer
- removed C11: 0.1uF, Capacitor_SMD:C_0603_1608Metric, symbol Device:C_Small
- removed C12: 330uF, Capacitor_SMD:CP_Elec_10x7.9, symbol Device:CP_Small
- removed C13: 22uF, Capacitor_SMD:C_0805_2012Metric, symbol Device:C_Small
- removed D4: (no value), Diode_SMD:Diode_Bridge_Vishay_DFS, symbol Device:D_Bridge_+-AA
- removed J2: Barrel_Jack_Switch, Connector_BarrelJack:BarrelJack_CUI_PJ-036AH-SMT_Horizontal, symbol Connector:Barrel_Jack_Switch
- removed P1, P2, P3: CONN_01X02, Pin_Headers:Pin_Header_Straight_1x02_Pitch2.54mm, symbol Connector_Generic:Conn_01x02
- removed P6: CONN_01X03, Pin_Headers:Pin_Header_Straight_1x03_Pitch2.00mm, symbol Connector_Generic:Conn_01x03
- removed Q1: NUD3124, Package_TO_SOT_SMD:SOT-23, symbol Power_Management-ML:NUD3124
- removed Q2: BCM857BS, Package_TO_SOT_SMD:SOT-363_SC-70-6, symbol Transistor_BJT-ML:BCM857BS
- removed Q3: DMG2305UX, Package_TO_SOT_SMD:SOT-23, symbol Transistor_FET-ML:DMG2305UX
- removed R2, R3: 3.9k, Resistor_SMD:R_0603_1608Metric, symbol Device:R
- removed R4: 1k, Resistor_SMD:R_0603_1608Metric, symbol Device:R
- removed R5: 4.7k, Resistor_SMD:R_0603_1608Metric, symbol Device:R
- removed R6: 47k, Resistor_SMD:R_0603_1608Metric, symbol Device:R
- removed R7: 10k, Resistor_SMD:R_0603_1608Metric, symbol Device:R
- removed R8: 44.2k, Resistor_SMD:R_0603_1608Metric, symbol Device:R
- removed R9: 232k, Resistor_SMD:R_0603_1608Metric, symbol Device:R
- removed SW1: Write, Button_Switch_SMD:SW_SPST_B3U-1000P, symbol Switch:SW_Push
- removed U5: AT24CS32, Package_DFN_QFN:DFN-8-1EP_3x2mm_P0.5mm_EP1.3x1.5mm, symbol Memory_EEPROM-ML:AT24CS32-MAHM
- removed U6: LMZ21700, Converter_DCDC-ML:Converter_DCDC_Texas-SIL0008E, symbol Converter_DCDC-ML:LMZ21700
- added C15, C16, C17: 0.33uF, Capacitor_SMD:C_0603_1608Metric, symbol Device:C_Small
- added C18, C19: 0.01uF, Capacitor_SMD:C_0603_1608Metric, symbol Device:C_Small
- added J1, J3, J4, J5: Screw_Terminal_01x02, TerminalBlock_Phoenix:TerminalBlock_Phoenix_PT-1,5-2-3.5-H_1x02_P3.50mm_Horizontal, symbol Connector:Screw_Terminal_01x02
- added J6: Screw_Terminal_01x03, TerminalBlock_Phoenix:TerminalBlock_Phoenix_PT-1,5-3-3.5-H_1x03_P3.50mm_Horizontal, symbol Connector:Screw_Terminal_01x03
- added J7: Screw_Terminal_01x04, TerminalBlock_Phoenix:TerminalBlock_Phoenix_PT-1,5-4-3.5-H_1x04_P3.50mm_Horizontal, symbol Connector:Screw_Terminal_01x04
- added U6: MAX3221CDBR, Package_SO:SSOP-16_5.3x6.2mm_P0.65mm, symbol Interface_UART:MAX3221
- added U7: ADuM1201ARZ, Package_SO:SOIC-8_3.9x4.9mm_P1.27mm, symbol Isolator:ADuM1201AR
- C14: value 3300pF -> 0.047uF; Description CAP, 0603, 3300pF, 5%, X7R, 10V -> CAP, 0603, .01uF, 10%, X7R, 50V; Manufacturer Vishay -> Murata Electronics; Part Number VJ0603Y332JXQPW1BC -> CC0603KRX7R9BB103; Tolerance 5% -> (none); Vendor Part Number 77-VJ0603Y332JXQPBC -> 603-CC603KRX7R9BB103; Voltage 10V -> (none)
- renumbered C16 to C1, C7 to C10, C3 to C11, C6 to C12, C9 to C13, C15 to C2, C10 to C3, C17 to C4, C2 to C5, C1 to C6, C5 to C7, C4 to C8, C8 to C9, J1 to J2, U7 to U1, U4 to U2, U1 to U3, U2 to U4, U3 to U5
Connections:
- net labels added: GEN5V, GENGND, GENIN, GENOUT, RXD, TXD
- net labels removed: +5VB, AC1, AC2, ALERT, ID_SC, ID_SD, VBulk
- wire segments 319 -> 268
- no-connect marks 0 -> 27
Other:
- note added: "Strapped for Normal Operation (Forced On)"
- note removed: "1."
- note removed: "5V Switcher"
- note removed: "Alert"
- note removed: "Hat ID EEPROM"
- note removed: "Ideal Diode"
- note removed: "Maximum Raspberry Pi current is 650mA."
- note removed: "Raspberry Pi can be safely back powered by this HAT."
- moved on the sheet: C1, C2, C3, C4, J2, R1, U1, U2

Commit message: PCB Version 3.0 files
Parts:
- added C20, C21: 2.2uF, Capacitor_SMD:C_0805_2012Metric, symbol Device:C_Small
- added F1: Polyfuse 1206L010/60WR 0.1A, Fuse:Fuse_1206_3216Metric_Pad1.42x1.75mm_HandSolder, symbol Device:Polyfuse
- added J8: Conn_02x06_Odd_Even, Connector_PinHeader_2.54mm:PinHeader_2x06_P2.54mm_Vertical, symbol Connector_Generic:Conn_02x06_Odd_Even
- added U8: MCP1754ST, Package_TO_SOT_SMD:SOT-89-3, symbol Regulator_Linear:MCP1754-3302E_SOT89
- U3: value MAX31850K -> MAX31850KATB; Part Number MAX31850KATB+ -> MAX31850KATB+T; Vendor Part Number 700-MAX31850KATB+ -> 700-MAX31850KATB+T
- U4, U5: value MAX31850K -> MAX31850KATB+T; Part Number MAX31850KATB+ -> MAX31850KATB+T; Vendor Part Number 700-MAX31850KATB+ -> 700-MAX31850KATB+T
- U7: value ADuM1201ARZ -> ADuM1201ARZ-RL7; mouser https://www.mouser.com/ProductDetail/Analog-Devices/ADUM1201ARZ?qs=sGAEpiMZZMssyD0wnx%2FymCCDPdsQyP%2F2CERA%2Fqc9nAY%3D -> https://www.mouser.com/ProductDetail/Analog-Devices/ADUM1201ARZ-RL7?qs=sGAEpiMZZMssyD0wnx%2FymCCDPdsQyP%2F22F9j%252BvOP7eI%3D
Connections:
- net +3.3VA: now also F1.2; no longer J6.1 (Pin_1)
- net GEN5V: now also C20.2, U8.1 (VI); no longer C16.2, C17.2, C18.1, U6.12 (FORCEON), U6.15 (VCC), U6.16 (~FORCEOFF), U7.1 (VDD1)
- net GENGND: no longer C18.2, J7.4 (Pin_4), U6.1 (~EN), U6.10 (~INVALID), U6.14 (GND), U7.4 (GND1)
- net GND: now also J8.1 (Pin_1), J8.11 (Pin_11), J8.3 (Pin_3), J8.5 (Pin_5), J8.7 (Pin_7), J8.9 (Pin_9)
- net GPIO23: now reaches J2.16 (GPIO23)
- net GPIO23: now also J8.2 (Pin_2)
- net GPIO24: now reaches J2.18 (GPIO24)
- net GPIO24: now also J8.4 (Pin_4)
- net GPIO9: now reaches J2.21 (GPIO09_SPI_MISO)
- net GPIO9: now also J8.10 (Pin_10)
- net GPIO25: now reaches J2.22 (GPIO25)
- net GPIO25: now also J8.6 (Pin_6)
- net GPIO8: now reaches J2.24 (GPIO08_SPI_CE0_N)
- net GPIO8: now also J8.8 (Pin_8)
- net GPIO7: now reaches J2.26 (GPIO07_SPI_CE1_N)
- net GPIO7: now also J8.12 (Pin_12)
- new net: F1.1, J6.1 (Pin_1)
- new net: C18.2, C20.1, C21.1, J7.4 (Pin_4), U6.1 (~EN), U6.10 (~INVALID), U6.14 (GND), U7.4 (GND1), U8.2 (GND)
- new net GEN3V3: C16.2, C17.2, C18.1, C21.2, U6.12 (FORCEON), U6.15 (VCC), U6.16 (~FORCEOFF), U7.1 (VDD1), U8.3 (VO)
- no-connect marks 27 -> 21
Other:
- note added: "Galvanic Isolation\nBoundary"
- note added: "Power"
- note added: "Strapped for Normal\nOperation (Forced On)"
- note removed: "Analog Power"
- note removed: "Strapped for Normal Operation (Forced On)"
- moved on the sheet: C14, C15, C16, C17, C18, C19, J7, U6, U7

Commit message: Candidate files for Version 3.1 of the PCB
Parts:
- added D20, D5: ASMT-RF45-AN002, LED_SMD:LED_0603_1608Metric, symbol Device:LED
- added D21: NSR20F30NXT5G, Diode_SMD:D_0603_1608Metric, symbol Device:D_Schottky
- added J9: Conn_01x04_Male, Connector_PinHeader_2.54mm:PinHeader_1x04_P2.54mm_Vertical, symbol Connector:Conn_01x04_Male
- added JP1, JP2: Jumper_NC_Small, Jumper:SolderJumper-2_P1.3mm_Bridged_RoundedPad1.0x1.5mm, symbol Device:Jumper_NC_Small
- added R10, R20: 120, Resistor_SMD:R_0603_1608Metric, symbol Device:R
- added R2, R3, R4, R5, R6, R7: 330, Resistor_SMD:R_0603_1608Metric, symbol Device:R
- added R8, R9: 4.7k, Resistor_SMD:R_0603_1608Metric, symbol Device:R
- C14: value 0.047uF -> 0.1uF; Description CAP, 0603, .01uF, 10%, X7R, 50V -> CAP, 0603, .1uF, 10%, X7R, 50V; Manufacturer Murata Electronics -> Yageo; Part Number CC0603KRX7R9BB103 -> CC0603KRX7R9BB104; Vendor Part Number 603-CC603KRX7R9BB103 -> 603-CC603KRX7R9BB104
- C15, C16, C17: value 0.33uF -> 0.1uF; Description CAP, 0603, .01uF, 10%, X7R, 50V -> CAP, 0603, .1uF, 10%, X7R, 50V; Manufacturer Murata Electronics -> Yageo; Part Number CC0603KRX7R9BB103 -> CC0603KRX7R9BB104; Vendor Part Number 603-CC603KRX7R9BB103 -> 603-CC603KRX7R9BB104
- F1: Description (none) -> FUSE, 1206, 100mA; Part Number (none) -> 1206L010/60WR; Vendor (none) -> Mouser; Vendor Part Number (none) -> 576-1206L010/60WR
- J1, J3, J4, J5: Description (none) -> Fixed Terminal Blocks PT 1.5/2-3.5H 2POS HRZ 3.5mm SCREW; Manufacturer (none) -> Phoenix Contact; Part Number (none) -> 1984617; Vendor (none) -> Mouser; Vendor Part Number (none) -> 651-1984617
- J6: Description (none) -> Fixed Terminal Blocks PT 1.5/3-3.5H 3POS HRZ 3.5mm SCREW; Manufacturer (none) -> Phoenix Contact; Part Number (none) -> 1984620; Vendor (none) -> Mouser; Vendor Part Number (none) -> 651-1984620
- J7: Description (none) -> Fixed Terminal Blocks PT 1.5/4-3.5H 4POS HRZ 3.5mm SCREW; Manufacturer (none) -> Phoenix Contact; Part Number (none) -> 1984633; Vendor (none) -> Mouser; Vendor Part Number (none) -> 651-1984633
- J8: Description (none) -> Headers & Wire Housings 06+06 DIL VERTICAL PIN HEADER GOLD+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; Manufacturer (none) -> Harwin; Part Number (none) -> M20-9760642; Vendor (none) -> Mouser; Vendor Part Number (none) -> 855-M20-9760642
- R1: Manufacturer Panasonic -> Yageo; Part Number ERJ-3EKF4701V -> AC0603FR-074K7L; Vendor Part Number 667-ERJ-3EKF4701V -> 603-AC0603FR-074K7L
- U2: value DS18S20 -> DS18B20; Part Number DS18S20+ -> DS18B20+; Vendor Part Number 700-DS18S20 -> 700-DS18B20+
- U3: value MAX31850KATB -> MAX31850KATB; Part Number MAX31850KATB+T -> MAX31850KATB+; Vendor Part Number 700-MAX31850KATB+T -> 700-MAX31850KATB+
- U4, U5: value MAX31850KATB+T -> MAX31850KATB; Part Number MAX31850KATB+T -> MAX31850KATB+; Vendor Part Number 700-MAX31850KATB+T -> 700-MAX31850KATB+
- U6: Description (none) -> IC, RS-232 Interface IC 1-Channel RS-232; Manufacturer (none) -> TI; Part Number (none) -> MAX3221CDBR; Vendor (none) -> Mouser; Vendor Part Number (none) -> 595-MAX3221CDBR
- U7: value ADuM1201ARZ-RL7 -> ADuM1201AR; Description (none) -> IC, Digital Isolators DUAL-CHANNEL DIGITAL ISOLATORS; Manufacturer (none) -> Analog Device; Part Number (none) -> ADUM1201AR; Vendor (none) -> Mouser; Vendor Part Number (none) -> 584-ADUM1201AR
Connections:
- net +3.3VA: now also JP1.2, JP2.2, R10.2
- net GEN5V: now also D21.1 (K); no longer J7.1 (Pin_1)
- net GENIN: now also U6.8 (RIN); no longer U6.11 (DIN)
- net GENOUT: now also U6.13 (DOUT); no longer U6.9 (ROUT)
- net GND: now also D5.1 (K), J9.1 (Pin_1)
- net GPIO23: now also R2.1; no longer J8.2 (Pin_2)
- net GPIO24: now also R3.1; no longer J8.4 (Pin_4)
- net GPIO25: now also R4.1; no longer J8.6 (Pin_6)
- net GPIO7: now also R7.1; no longer J8.12 (Pin_12)
- net GPIO8: now also R5.1; no longer J8.8 (Pin_8)
- net GPIO9: now also R6.1; no longer J8.10 (Pin_10)
- net RXD: no longer J2.10 (GPIO15_RXD0), U7.6 (VOB)
- net SDA: now reaches J2.3 (GPIO02_SDA1_I2C)
- net SDA: now also J9.3 (Pin_3), R9.1
- net SCL: now reaches J2.5 (GPIO03_SCL1_I2C)
- net SCL: now also J9.4 (Pin_4), R8.1
- net 3V3FUSED: now reaches F1.1, J6.1 (Pin_1)
- net 3V3FUSED: now also J9.2 (Pin_2)
- net GEN-OUT-TTL: now reaches U7.2 (VOA)
- net GEN-OUT-TTL: now also U6.11 (DIN); no longer U6.8 (RIN)
- net GEN-IN-TTL: now reaches U7.3 (VIB)
- net GEN-IN-TTL: now also U6.9 (ROUT); no longer U6.13 (DOUT)
- net GNDD: now reaches C18.2, C20.1, C21.1, J7.4 (Pin_4), U6.1 (~EN), U6.10 (~INVALID), U6.14 (GND), U7.4 (GND1), U8.2 (GND)
- net GNDD: now also D20.1 (K)
- net GEN3V3 renamed +3V3
- net +3V3: now also R20.2
- new net: J2.10 (GPIO15_RXD0), U7.6 (VOB)
- new net: D21.2 (A), J7.1 (Pin_1)
- new net: J8.2 (Pin_2), R2.2
- new net: J8.4 (Pin_4), R3.2
- new net: J8.6 (Pin_6), R4.2
- new net: J8.8 (Pin_8), R5.2
- new net: J8.10 (Pin_10), R6.2
- new net: J8.12 (Pin_12), R7.2
- new net: JP1.1, R8.2
- new net: JP2.1, R9.2
- new net: D20.2 (A), R20.1
- new net: D5.2 (A), R10.1
- no-connect marks 21 -> 19
Other:
- note added: "Current limiting resistors for external LED\ndriven from RPi GPIO outputs. Season to \ntaste. RPi GPIO can supply approx 8mA.\n"
- note added: "Green"
- note added: "Strapped for \nNormal Operation\n(Forced On)"
- note removed: "Strapped for Normal\nOperation (Forced On)"
- moved on the sheet: C1, C14, C15, C16, C17, C18, C19, C2, C4, F1, J1, J2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

Commit message: delete unneeded component metadata
Parts:
- F1: Mouser 576-1206L010/60WR -> (none)
- U7: mouser https://www.mouser.com/ProductDetail/Analog-Devices/ADUM120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 -> (none)
Changed lines of the file:
@@
 F 2 "Fuse:Fuse_1206_3216Metric_Pad1.42x1.75mm_HandSolder" H 8550 5600 50  0001 L CNN
 F 3 "https://www.mouser.com/datasheet/2/240/Littelfuse_PTC_1206L_Datasheet.pdf-477012.pdf" H 8500 5800 50  0001 C CNN
-F 4 "576-1206L010/60WR" V 8500 5800 50  0001 C CNN "Mouser"
-F 5 " 1206L010/60WR " H 8500 5800 50  0001 C CNN "Part Number"
-F 6 "576-1206L010/60WR" H 8500 5800 50  0001 C CNN "Vendor Part Number"
-F 7 "FUSE, 1206,  100mA" H 8500 5800 50  0001 C CNN "Description"
-F 8 "Mouser" H 8500 5800 50  0001 C CNN "Vendor"
+F 4 " 1206L010/60WR " H 8500 5800 50  0001 C CNN "Part Number"
+F 5 "576-1206L010/60WR" H 8500 5800 50  0001 C CNN "Vendor Part Number"
+F 6 "FUSE, 1206,  100mA" H 8500 5800 50  0001 C CNN "Description"
+F 7 "Mouser" H 8500 5800 50  0001 C CNN "Vendor"
 	1    8500 5800
 	0    1    1    0
@@
 F 2 "Package_SO:SOIC-8_3.9x4.9mm_P1.27mm" H 4550 6250 50  0001 C CIN
 F 3 "https://www.mouser.com/datasheet/2/609/ADuM1200_1201-279454.pdf" H 4550 6550 50  0001 C CNN
-F 4 "https://www.mouser.com/ProductDetail/Analog-Devices/ADUM1201ARZ-RL7?qs=sGAEpiMZZMssyD0wnx%2FymCCDPdsQyP%2F22F9j%252BvOP7eI%3D" H 4550 6650 50  0001 C CNN "mouser"
-F 5 "IC, Digital Isolators DUAL-CHANNEL DIGITAL ISOLATORS " H 4550 6650 50  0001 C CNN "Description"
-F 6 "Analog Device" H 4550 6650 50  0001 C CNN "Manufacturer"
-F 7 "ADUM1201AR" H 4550 6650 50  0001 C CNN "Part Number"
-F 8 "Mouser" H 4550 6650 50  0001 C CNN "Vendor"
-F 9 "584-ADUM1201AR" H 4550 6650 50  0001 C CNN "Vendor Part Number"
+F 4 "IC, Digital Isolators DUAL-CHANNEL DIGITAL ISOLATORS " H 4550 6650 50  0001 C CNN "Description"
+F 5 "Analog Device" H 4550 6650 50  0001 C CNN "Manufacturer"
+F 6 "ADUM1201AR" H 4550 6650 50  0001 C CNN "Part Number"
+F 7 "Mouser" H 4550 6650 50  0001 C CNN "Vendor"
+F 8 "584-ADUM1201AR" H 4550 6650 50  0001 C CNN "Vendor Part Number"
 	1    4550 6650
 	1    0    0    -1

Commit message: add some LCSC part numbers
Parts:
- C1, C2, C20, C21: LCSC (none) -> C49217
- C10, C11, C12, C13, C14, C15, C16, C17, C3, C6, C8: LCSC (none) -> C14663
- C18, C19, C5, C7, C9: LCSC (none) -> C57112
- C4: LCSC (none) -> C45783
- D1, D2, D3: LCSC (none) -> C252430
- D20, D5: LCSC (none) -> C72043
- D21: LCSC (none) -> C8598
- F1: LCSC (none) -> C261947
- FB1, FB2, FB3, FB4, FB5, FB6: LCSC (none) -> C73100
- R1, R8, R9: LCSC (none) -> C23162
- R10, R20: LCSC (none) -> C22787
- R2, R3, R4, R5, R6, R7: LCSC (none) -> C23138
- U1, U8: LCSC (none) -> C6186
- U6: LCSC (none) -> C105243
- U7: LCSC (none) -> C9669
